File: OmniStimEvalBoard.kicad_sch (KiCad schematic)
At the start: 6 parts

Commit message: Additional Rev 2 changes done
Connections:
- net ESP32-S2/ESP_ADC2_CH9 renamed ESP32-S2/ESP_ADC2_CH8
Other:
- sheet Development Extras ports: added ESP_UDB_DP, ESP_USB_DN; removed none
- sheet ESP32-S2 ports: added ESP_ADC2_CH8, USB_D+, USB_D-; removed ESP_ADC2_CH9
Changed lines of the file:
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@@
+	(wire
+		(pts
+			(xy 17.78 101.6) (xy 35.56 101.6)
+		)
+		(stroke
+			(width 0)
+			(type default)
+		)
+	)
 	(wire
 		(pts
@@
 	(wire
 		(pts
+			(xy 35.56 41.91) (xy 15.24 41.91)
+		)
+		(stroke
+			(width 0)
+			(type default)
+		)
+	)
+	(wire
+		(pts
 			(xy 25.4 52.07) (xy 25.4 93.98)
 		)
@@
 	(wire
 		(pts
+			(xy 15.24 104.14) (xy 35.56 104.14)
+		)
+		(stroke
+			(width 0)
+			(type default)
+		)
+	)
+	(wire
+		(pts
 			(xy 93.98 57.15) (xy 100.33 57.15)
 		)
@@
 	(wire
 		(pts
+			(xy 17.78 44.45) (xy 17.78 101.6)
+		)
+		(stroke
+			(width 0)
+			(type default)
+		)
+	)
+	(wire
+		(pts
 			(xy 25.4 93.98) (xy 35.56 93.98)
 		)
@@
 	(wire
 		(pts
+			(xy 35.56 44.45) (xy 17.78 44.45)
+		)
+		(stroke
+			(width 0)
+			(type default)
+		)
+	)
+	(wire
+		(pts
 			(xy 35.56 49.53) (xy 22.86 49.53)
 		)
@@
 		(pts
 			(xy 190.5 50.8) (xy 190.5 63.5)
+		)
+		(stroke
+			(width 0)
+			(type default)
+		)
+	)
+	(wire
+		(pts
+			(xy 15.24 41.91) (xy 15.24 104.14)
 		)
 		(stroke
@@
 	(sheet
 		(at 35.56 80.01)
-		(size 35.56 21.59)
+		(size 35.56 25.4)
 		(exclude_from_sim no)
 		(in_bom yes)
@@
 		)
 		(property "Sheetfile" "devextras.kicad_sch"
-			(at 35.56 102.1846 0)
+			(at 35.56 105.9946 0)
 			(effects
 				(font
@@
 				)
 				(justify right)
+			)
+		)
+		(pin "ESP_UDB_DP" input
+			(at 35.56 101.6 180)
+			(effects
+				(font
+					(size 1.27 1.27)
+				)
+				(justify left)
+			)
+		)
+		(pin "ESP_USB_DN" input
+			(at 35.56 104.14 180)
+			(effects
+				(font
+					(size 1.27 1.27)
+				)
+				(justify left)
 			)
 		)
@@
 			)
 		)
-		(pin "ESP_ADC2_CH9" input
+		(pin "ESP_ADC2_CH8" input
 			(at 85.09 26.67 0)
 			(effects
@@
 			)
 		)
+		(pin "USB_D+" input
+			(at 35.56 44.45 180)
+			(effects
+				(font
+					(size 1.27 1.27)
+				)
+				(justify left)
+			)
+		)
+		(pin "USB_D-" input
+			(at 35.56 41.91 180)
+			(effects
+				(font
+					(size 1.27 1.27)
+				)
+				(justify left)
+			)
+		)
