File: devextras.kicad_sch (KiCad schematic)
At the start: 30 parts, among them Q601 L8050QLT1G, Q602 L8050QLT1G, SW601 TS-1088-AR02016, SW602 TS-1088-AR02016, U601 AMS1117-3.3, U602 CP2102N-A02-GQFN28R

Commit message: rev 2 errata resolved
Connections:
- net ESP_EN: now also H601.2
- net ESP_IO0 : now also H601.4
- net GND: no longer H601.2, H601.4
- net UART_RX: now also U602.26 (TXD); no longer U602.25 (RXD)
- net UART_TX: now also U602.25 (RXD); no longer U602.26 (TXD)
Other:
- moved on the sheet: H601
Changed lines of the file:
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@@
 	)
 	(junction
-		(at 54.61 156.21)
-		(diameter 0)
-		(color 0 0 0 0)
-	)
-	(junction
 		(at 151.13 102.87)
 		(diameter 0)
@@
 	)
 	(junction
-		(at 54.61 158.75)
-		(diameter 0)
-		(color 0 0 0 0)
-	)
-	(junction
 		(at 49.53 71.12)
 		(diameter 0)
@@
 	(wire
 		(pts
-			(xy 54.61 156.21) (xy 54.61 158.75)
-		)
-		(stroke
-			(width 0)
-			(type default)
-		)
-	)
-	(wire
-		(pts
 			(xy 151.13 77.47) (xy 151.13 102.87)
 		)
@@
 	(wire
 		(pts
-			(xy 54.61 158.75) (xy 54.61 161.29)
-		)
-		(stroke
-			(width 0)
-			(type default)
-		)
-	)
-	(wire
-		(pts
 			(xy 151.13 67.31) (xy 151.13 77.47)
 		)
@@
 	(wire
 		(pts
-			(xy 54.61 153.67) (xy 54.61 156.21)
-		)
-		(stroke
-			(width 0)
-			(type default)
-		)
-	)
-	(wire
-		(pts
 			(xy 44.45 71.12) (xy 46.99 71.12)
 		)
@@
 		)
 	)
+	(hierarchical_label "UART_RX"
+		(shape input)
+		(at 203.2 36.83 0)
+		(effects
+			(font
+				(size 1.27 1.27)
+			)
+			(justify left)
+		)
+	)
 	(hierarchical_label "UART_TX"
 		(shape input)
-		(at 44.45 153.67 180)
+		(at 36.83 153.67 180)
 		(effects
 			(font
@@
 	(hierarchical_label "UART_TX"
 		(shape input)
-		(at 203.2 36.83 0)
+		(at 203.2 39.37 0)
 		(effects
 			(font
@@
 		)
 	)
-	(hierarchical_label "UART_RX"
+	(hierarchical_label "ESP_IO0 "
 		(shape input)
-		(at 203.2 39.37 0)
+		(at 46.99 156.21 0)
 		(effects
 			(font
@@
 		)
 	)
+	(hierarchical_label "ESP_EN"
+		(shape input)
+		(at 46.99 153.67 0)
+		(effects
+			(font
+				(size 1.27 1.27)
+			)
+			(justify left)
+		)
+	)
 	(hierarchical_label "ESP_IO0 "
 		(shape input)
@@
 	(hierarchical_label "UART_RX"
 		(shape input)
-		(at 44.45 156.21 180)
+		(at 36.83 156.21 180)
 		(effects
 			(font
@@
 	(symbol
 		(lib_id "power:+3V3")
-		(at 44.45 158.75 90)
+		(at 36.83 158.75 90)
 		(unit 1)
 		(exclude_from_sim no)
@@
 		(fields_autoplaced yes)
 		(property "Reference" "#PWR0601"
-			(at 48.26 158.75 0)
+			(at 40.64 158.75 0)
 			(effects
 				(font
@@
 		)
 		(property "Value" "+3V3"
-			(at 40.64 158.7499 90)
+			(at 33.02 158.7499 90)
 			(effects
 				(font
@@
 		)
 		(property "Footprint" ""
-			(at 44.45 158.75 0)
+			(at 36.83 158.75 0)
 			(effects
 				(font
@@
 		)
 		(property "Datasheet" ""
-			(at 44.45 158.75 0)
+			(at 36.83 158.75 0)
 			(effects
 				(font
@@
 		)
 		(property "Description" "Power symbol creates a global label with name \"+3V3\""
-			(at 44.45 158.75 0)
+			(at 36.83 158.75 0)
 			(effects
 				(font
@@
 	(symbol
 		(lib_id "power:GND")
-		(at 54.61 161.29 0)
+		(at 46.99 158.75 0)
 		(unit 1)
 		(exclude_from_sim no)
@@
 		(fields_autoplaced yes)
 		(property "Reference" "#PWR0602"
-			(at 54.61 167.64 0)
+			(at 46.99 165.1 0)
 			(effects
 				(font
@@
 		)
 		(property "Value" "GND"
-			(at 54.61 166.37 0)
+			(at 46.99 163.83 0)
 			(effects
 				(font
@@
 		)
 		(property "Footprint" ""
-			(at 54.61 161.29 0)
+			(at 46.99 158.75 0)
 			(effects
 				(font
@@
 		)
 		(property "Datasheet" ""
-			(at 54.61 161.29 0)
+			(at 46.99 158.75 0)
 			(effects
 				(font
@@
 		)
 		(property "Description" "Power symbol creates a global label with name \"GND\" , ground"
-			(at 54.61 161.29 0)
+			(at 46.99 158.75 0)
 			(effects
 				(font
@@
 	(symbol
 		(lib_id "easyeda2kicad:PZ254-2-03-S")
-		(at 49.53 156.21 0)
+		(at 41.91 156.21 0)
 		(unit 1)
 		(exclude_from_sim no)
@@
 		(fields_autoplaced yes)
 		(property "Reference" "H601"
-			(at 49.53 146.05 0)
+			(at 41.91 146.05 0)
 			(effects
 				(font
@@
 		)
 		(property "Value" "PZ254-2-03-S"
-			(at 49.53 148.59 0)
+			(at 41.91 148.59 0)
 			(effects
 				(font
@@
 		)
 		(property "Footprint" "easyeda2kicad:HDR-SMD_6P-P2.54-V-M-R2-C3-LS7.5-2"
-			(at 49.53 166.37 0)
+			(at 41.91 166.37 0)
 			(effects
 				(font
@@
 		)
 		(property "Datasheet" "https://www.lcsc.com/product-detail/Pin-Headers_HCTL-PZ254-2-03-S_C3294461.html"
-			(at 49.53 156.21 0)
+			(at 41.91 156.21 0)
 			(effects
 				(font
@@
 		)
 		(property "Description" ""
-			(at 49.53 156.21 0)
+			(at 41.91 156.21 0)
 			(effects
 				(font
@@
 		)
 		(property "LCSC Part" "C3294461"
-			(at 49.53 168.91 0)
+			(at 41.91 168.91 0)
 			(effects
 				(font
@@
 		)
 		(property "MPN" "PZ254-2-03-S"
-			(at 49.53 156.21 0)
+			(at 41.91 156.21 0)
 			(effects
 				(font

Commit message: Additional Rev 2 changes done
Parts:
- added LED602, LED603: RED LED, easyeda2kicad:LED0805-R-RD, symbol easyeda2kicad:FC-2012HRK-620D
- added R602, R604, R610, R613: 5.1K, easyeda2kicad:R0603, symbol easyeda2kicad:RC0603FR-075K1L
- added USB602: TYPEC-304YSSW-ACP16, easyeda2kicad:USB-SMD_TYPEC-304YSSW-ACP16, symbol easyeda2kicad:TYPEC-304YSSW-ACP16
- LED601: value FC-2012HRK-620D -> RED LED
- renumbered R602 to R603, R604 to R605, R605 to R606, R606 to R607, R603 to R608, R607 to R609, R608 to R611, R609 to R612, R610 to R614, R611 to R615
Connections:
- net +3V3: now also R610.2, R613.2
- net GND: now also R602.1, R604.1, USB602.13 (GND), USB602.14 (GND), USB602.15 (GND), USB602.16 (GND), USB602.A1B12 (GND), USB602.B1A12 (GND)
- net USB_VBUS: now also USB602.A4B9 (VBUS), USB602.B4A9 (VBUS)
- net RXT: now reaches U602.18 (GPIO.1/RXT)
- net RXT: now also LED603.2 (-)
- net TXT: now reaches U602.19 (GPIO.0/TXT)
- net TXT: now also LED602.2 (-)
- new net: LED603.1 (+), R613.1
- new net: LED602.1 (+), R610.1
- new net: R602.2, USB602.A5 (CC1)
- new net: R604.2, USB602.B5 (CC2)
- new net ESP_UDB_DP: USB602.A6 (DP1), USB602.B6 (DP2)
- new net ESP_USB_DN: USB602.A7 (DN1), USB602.B7 (DN2)
Other:
- moved on the sheet: C601, C602, C603, C604, D601, H601, H602, LED601, R608, U601
