File: esp32s2.kicad_sch (KiCad schematic)
At the start: 6 parts, among them U201 ESP32-S2-MINI-2-N4

Commit message: Additional Rev 2 changes done
Parts:
- added TP201: APLL, TestPoint:TestPoint_Pad_1.0x1.0mm, symbol Connector:TestPoint
Connections:
- net ESP_APLL_OUT: now also TP201.1
- net USB_D-: now reaches U201.23 (IO19)
- net ESP_ADC2_CH8: now reaches U201.25 (IO21)
- net ESP_ADC2_CH9 renamed USB_D+
Changed lines of the file:
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@@
+	)
+	(junction
+		(at 90.17 109.22)
+		(diameter 0)
+		(color 0 0 0 0)
 	)
 	(junction
@@
 	(wire
 		(pts
+			(xy 86.36 109.22) (xy 90.17 109.22)
+		)
+		(stroke
+			(width 0)
+			(type default)
+		)
+	)
+	(wire
+		(pts
 			(xy 130.81 139.7) (xy 133.35 139.7)
 		)
@@
 	(wire
 		(pts
+			(xy 90.17 109.22) (xy 101.6 109.22)
+		)
+		(stroke
+			(width 0)
+			(type default)
+		)
+	)
+	(wire
+		(pts
 			(xy 158.75 139.7) (xy 161.29 139.7)
 		)
@@
 		)
 	)
+	(hierarchical_label "ESP_ADC2_CH8"
+		(shape input)
+		(at 101.6 119.38 180)
+		(effects
+			(font
+				(size 1.27 1.27)
+			)
+			(justify right)
+		)
+	)
 	(hierarchical_label "TXD0"
 		(shape input)
@@
 	(hierarchical_label "ESP_APLL_OUT"
 		(shape input)
-		(at 101.6 109.22 180)
+		(at 86.36 109.22 180)
 		(effects
 			(font
@@
 		)
 	)
+	(hierarchical_label "USB_D-"
+		(shape input)
+		(at 101.6 114.3 180)
+		(effects
+			(font
+				(size 1.27 1.27)
+			)
+			(justify right)
+		)
+	)
 	(hierarchical_label "GPIO_DAC_LDAC"
 		(shape input)
@@
 		)
 	)
-	(hierarchical_label "ESP_ADC2_CH9"
+	(hierarchical_label "USB_D+"
 		(shape input)
 		(at 101.6 116.84 180)
@@
 					(unit 1)
 				)
+			)
+		)
+	)
+	(symbol
+		(lib_id "Connector:TestPoint")
+		(at 90.17 109.22 0)
+		(unit 1)
+		(exclude_from_sim no)
+		(in_bom yes)
+		(on_board yes)
+		(dnp no)
+		(fields_autoplaced yes)
+		(property "Reference" "TP201"
+			(at 92.71 104.6479 0)
+			(effects
+				(font
+					(size 1.27 1.27)
+				)
+				(justify left)
+			)
+		)
+		(property "Value" "APLL"
+			(at 92.71 107.1879 0)
+			(effects
+				(font
+					(size 1.27 1.27)
+				)
+				(justify left)
+			)
+		)
+		(property "Footprint" "TestPoint:TestPoint_Pad_1.0x1.0mm"
+			(at 95.25 109.22 0)
+			(effects
+				(font
+					(size 1.27 1.27)
+				)
+				(hide yes)
+			)
+		)
+		(property "Datasheet" "~"
+			(at 95.25 109.22 0)
+			(effects
+				(font
+					(size 1.27 1.27)
+				)
+				(hide yes)
+			)
+		)
+		(property "Description" "test point"
+			(at 90.17 109.22 0)
+			(effects
+				(font
+					(size 1.27 1.27)
+				)
+				(hide yes)
+			)
+		)
+		(pin "1"
+		)
+		(instances
+			(project ""
+				(path "/3f793f1c-3d2c-449d-8c79-5d2783def882/d0bf1820-e0f9-4ed8-8e96-40c0d535d7f1"
+					(reference "TP201")
+					(unit 1)
+				)
