File: coarsecap.kicad_sch (KiCad schematic)
At the start: 14 parts, among them SW801 DSHP04TS-S, SW802 DSHP04TS-S

Commit message: Starting work on OmniStimDriverBoard design
Parts:
- removed SW801, SW802: DSHP04TS-S, easyeda2kicad:SW-SMD_8P-L6.7-W5.4-P1.27-LS8.5, symbol easyeda2kicad:DSHP04TS-S
- added K801, K802, K803, K804, K805, K806, K807: G6K-2F-Y-DC5, easyeda2kicad:RELAY-SMD_G6K-2F-X-XX, symbol easyeda2kicad:G6K-2F-Y-DC5
